Commit message: Ajout de navigation autonome (non fonctionnel), modification du fichier URDF

File: urdf/camera.urdf.xacro (robot description, xacro)
@@ -101,5 +101,5 @@
         <alwaysOn>true</alwaysOn>
         <updateRate>0.0</updateRate>
-        <cameraName>stereo</cameraName>
+        <cameraName>stereo_camera</cameraName>
         <imageTopicName>image_raw</imageTopicName>
         <cameraInfoTopicName>camera_info</cameraInfoTopicName>
@@ -122,3 +122,13 @@
     <material>Gazebo/Black</material>
   </gazebo>
+  <gazebo>
+    <plugin name="imu_plugin" filename="libgazebo_ros_imu.so">
+      <alwaysOn>true</alwaysOn>
+      <bodyName>camera_left_link</bodyName>
+      <topicName>imu</topicName>
+      <serviceName>imu_service</serviceName>
+      <gaussianNoise>0.0</gaussianNoise>
+      <updateRate>20.0</updateRate>
+    </plugin>
+  </gazebo>
 </robot>

File: urdf/suspensions_wheels.urdf.xacro (robot description, xacro)
@@ -110,4 +110,28 @@
       <child link="${prefix}_rocker1"/>
       <origin xyz="0 ${reflect*bodywidth/2} 0" />
+      <!-- <axis xyz="0 1 0" rpy="0 0 0" />
+      joint torsional spring plugin <axis>
+        <limit>
+          <lower>-0.1</lower>
+          <upper>0.1</upper>
+        </limit>
+        <dynamics>
+          <spring_stiffness>2500</spring_stiffness>
+          <spring_reference>0.06</spring_reference>
+          <damping>20.0</damping>
+          <friction>0.75</friction>
+        </dynamics>
+        <use_parent_model_frame>0</use_parent_model_frame>
+      </axis>
+      <physics>
+        <ode>
+          <implicit_spring_damper>1</implicit_spring_damper>
+          <cfm_damping>1</cfm_damping>
+          <limit>
+            <cfm>0</cfm>
+            <erp>0.2</erp>
+          </limit>
+        </ode>
+      </physics> -->
     </joint>
     <link name="${prefix}_rocker2">

Commit message: Avancement localization - Non fonctionnel

File: urdf/camera.urdf.xacro (robot description, xacro)
@@ -64,9 +64,9 @@
       <update_rate>30.0</update_rate>
       <camera name="left">
-        <horizontal_fov>1.3962634</horizontal_fov>
         <image>
-          <width>800</width>
-          <height>800</height>
+          <width>1280</width>
+          <height>720</height>
           <format>R8G8B8</format>
+          <hfov>110</hfov>
         </image>
         <clip>
@@ -82,8 +82,8 @@
       <camera name="right">
         <pose>0 -0.16 0 0 0 0</pose>
-        <horizontal_fov>1.3962634</horizontal_fov>
         <image>
-          <width>800</width>
-          <height>800</height>
+          <width>1280</width>
+          <height>720</height>
+          <hfov>110</hfov>
           <format>R8G8B8</format>
         </image>
@@ -126,5 +126,5 @@
       <alwaysOn>true</alwaysOn>
       <bodyName>camera_left_link</bodyName>
-      <topicName>imu</topicName>
+      <topicName>imu/data</topicName>
       <serviceName>imu_service</serviceName>
       <gaussianNoise>0.0</gaussianNoise>

File: urdf/gps.urdf.xacro (robot description, xacro)
@@ -66,4 +66,15 @@
 <!--                <velocityGaussianNoise>0.05 0.05 0.05</velocityGaussianNoise>-->
 	</plugin>
+	<!-- Ground truth plugin -->
+	<plugin name="p3d_base_controller" filename="libgazebo_ros_p3d.so">
+      <alwaysOn>true</alwaysOn>
+      <updateRate>200.0</updateRate>
+      <bodyName>base_link</bodyName>
+      <topicName>ground_truth/state</topicName>
+      <gaussianNoise>0.0</gaussianNoise>
+      <frameName>map</frameName>
+      <xyzOffsets>0 0 0</xyzOffsets>
+      <rpyOffsets>0 0 0</rpyOffsets>
+    </plugin>
 </gazebo>
  <gazebo reference="GPS_Beacon">

File: urdf/rover1.urdf.xacro (robot description, xacro)
@@ -1,7 +1,7 @@
 <?xml version="1.0"?>
 <robot name="paul" xmlns:xacro="http://ros.org/wiki/xacro">
-  <xacro:property name="bodywidth" value="0.5" />
+  <xacro:property name="bodywidth" value="1" />
   <xacro:property name="bodylen" value="1" />
-  <xacro:property name="bodyhei" value="0.2" />
+  <xacro:property name="bodyhei" value="0.3" />
   <xacro:property name="wheeldiam" value="0.254" />
   <xacro:property name="wheellen" value="0.002" />
@@ -48,8 +48,9 @@
       </geometry>
     </collision>
-     <xacro:default_inertial mass="30"/>
+     <xacro:default_inertial mass="46"/>
   </link>
 <!-- Insert Suspensions and wheels -->
- <xacro:include filename="$(find polyorbite_rover)/urdf/suspensions_wheels.urdf.xacro"/>
+<xacro:include filename="$(find polyorbite_rover)/urdf/suspensions_wheels.urdf.xacro"/>
+<!-- <xacro:include filename="$(find polyorbite_rover)/bash/fileMaker/suspension_wheels.urdf.xacro"/>-->
 <!-- Insert Camera -->
  <xacro:include filename="$(find polyorbite_rover)/urdf/camera.urdf.xacro"/>

File: urdf/suspensions_wheels.urdf.xacro (robot description, xacro)
@@ -15,5 +15,5 @@
           <cylinder radius="${wheeldiam/2}" length="0.1"/>
         </geometry>
-      </collision>
+       </collision>
       <xacro:default_inertial mass="1"/>
     </link>
@@ -30,12 +30,15 @@
       </actuator>
       <joint name="${prefix}_${suffix}_wheel_joint">
-        <hardwareInterface>VelocityJointInterface</hardwareInterface>
+        <!--<hardwareInterface>hardware_interface/EffortJointInterface</hardwareInterface>-->
+        <hardwareInterface>hardware_interface/VelocityJointInterface</hardwareInterface>
       </joint>
     </transmission>
     <gazebo reference="${prefix}_${suffix}_wheel">
-      <mu1 value="200.0"/>
-      <mu2 value="100.0"/>
-      <kp value="10000000.0" />
-      <kd value="1.0" />
+	  <mu1 value="100.0"/>
+      <mu2 value="200.0"/>
+      <kp value="1000000.0" />
+      <kd value="100.0" />
+      <!--<maxVel>1.0</maxVel>-->
+	  <minDepth>0.005</minDepth>
       <material>Gazebo/Grey</material>
     </gazebo>
