Commit message: Ajout camera et streaming module

File: urdf/rover1.urdf.xacro (robot description, xacro)
@@ -185,4 +185,71 @@
   <xacro:rocker prefix="right" reflect="-1" />
   <xacro:rocker prefix="left" reflect="1" />
+  <joint name="camera_joint" type="fixed">
+    <axis xyz="0 1 0" />
+    <origin xyz="${bodylen/2} 0 0" rpy="0 0 0"/>
+    <parent link="base_link"/>
+    <child link="camera_link"/>
+  </joint>
+  <!-- Camera -->
+  <link name="camera_link">
+    <collision>
+      <origin xyz="0 0 0" rpy="0 0 0"/>
+      <geometry>
+    <box size="0.03 0.175 0.033"/>
+      </geometry>
+    </collision>
+    <visual>
+      <origin xyz="0 0 0" rpy="0 0 0"/>
+      <geometry>
+    <box size="0.03 0.175 0.033"/>
+      </geometry>
+      <material name="red"/>
+    </visual>
+    <inertial>
+      <mass value="0.166" />
+      <origin xyz="0 0 0" rpy="0 0 0"/>
+      <inertia ixx="1e-6" ixy="0" ixz="0" iyy="1e-6" iyz="0" izz="1e-6" />
+    </inertial>
+  </link>
+  <!-- camera -->
+  <gazebo reference="camera_link">
+    <sensor type="camera" name="camera1">
+      <update_rate>30.0</update_rate>
+      <camera name="head">
+        <horizontal_fov>1.3962634</horizontal_fov>
+        <image>
+          <width>800</width>
+          <height>800</height>
+          <format>R8G8B8</format>
+        </image>
+        <clip>
+          <near>0.02</near>
+          <far>300</far>
+        </clip>
+        <noise>
+          <type>gaussian</type>
+          <!-- Noise is sampled independently per pixel on each frame.
+               That pixel's noise value is added to each of its color
+               channels, which at that point lie in the range [0,1]. -->
+          <mean>0.0</mean>
+          <stddev>0.007</stddev>
+        </noise>
+      </camera>
+      <plugin name="camera_controller" filename="libgazebo_ros_camera.so">
+        <alwaysOn>true</alwaysOn>
+        <updateRate>0.0</updateRate>
+        <cameraName>rrbot/camera1</cameraName>
+        <imageTopicName>image_raw</imageTopicName>
+        <cameraInfoTopicName>camera_info</cameraInfoTopicName>
+        <frameName>camera_link</frameName>
+        <hackBaseline>0.07</hackBaseline>
+        <distortionK1>0.0</distortionK1>
+        <distortionK2>0.0</distortionK2>
+        <distortionK3>0.0</distortionK3>
+        <distortionT1>0.0</distortionT1>
+        <distortionT2>0.0</distortionT2>
+      </plugin>
+    </sensor>
+  </gazebo>
   <gazebo>
     <plugin name="gazebo_ros_control" filename="libgazebo_ros_control.so">

Commit message: Added Camera controller, now functionnal with RVIZ visualisation

File: urdf/rover1.urdf.xacro (robot description, xacro)
@@ -185,12 +185,12 @@
   <xacro:rocker prefix="right" reflect="-1" />
   <xacro:rocker prefix="left" reflect="1" />
-  <joint name="camera_joint" type="fixed">
+  <joint name="camera_base_joint" type="fixed">
     <axis xyz="0 1 0" />
     <origin xyz="${bodylen/2} 0 0" rpy="0 0 0"/>
     <parent link="base_link"/>
-    <child link="camera_link"/>
+    <child link="camera_base_link"/>
   </joint>
-  <!-- Camera -->
-  <link name="camera_link">
+  <!-- Camera base-->
+  <link name="camera_base_link">
     <collision>
       <origin xyz="0 0 0" rpy="0 0 0"/>
@@ -203,4 +203,32 @@
       <geometry>
     <box size="0.03 0.175 0.033"/>
+      </geometry>
+      <material name="black"/>
+    </visual>
+    <inertial>
+      <mass value="0.166" />
+      <origin xyz="0 0 0" rpy="0 0 0"/>
+      <inertia ixx="1e-6" ixy="0" ixz="0" iyy="1e-6" iyz="0" izz="1e-6" />
+    </inertial>
+  </link>
+  <!-- Camera -->
+<xacro:macro name="Zedcamera" params="prefix reflect">
+  <joint name="camera_${prefix}_joint" type="fixed">
+    <axis xyz="0 1 0" />
+    <origin xyz="0.015 ${reflect*0.08} 0" rpy="0 0 0"/>
+    <parent link="camera_base_link"/>
+    <child link="camera_${prefix}_link"/>
+  </joint>
+  <link name="camera_${prefix}_link">
+    <collision>
+      <origin xyz="0 0 0" rpy="0 0 0"/>
+      <geometry>
+    <box size="0.01 0.01 0.01"/>
+      </geometry>
+    </collision>
+    <visual>
+      <origin xyz="0 0 0" rpy="0 0 0"/>
+      <geometry>
+    <box size="0.01 0.01 0.01"/>
       </geometry>
       <material name="red"/>
@@ -212,9 +240,12 @@
     </inertial>
   </link>
+ </xacro:macro>
+  <xacro:Zedcamera prefix="right" reflect="-1" />
+  <xacro:Zedcamera prefix="left" reflect="1" />
   <!-- camera -->
-  <gazebo reference="camera_link">
-    <sensor type="camera" name="camera1">
+  <gazebo reference="camera_left_link">
+    <sensor type="multicamera" name="stereo_camera">
       <update_rate>30.0</update_rate>
-      <camera name="head">
+      <camera name="left">
         <horizontal_fov>1.3962634</horizontal_fov>
         <image>
@@ -229,19 +260,35 @@
         <noise>
           <type>gaussian</type>
-          <!-- Noise is sampled independently per pixel on each frame.
-               That pixel's noise value is added to each of its color
-               channels, which at that point lie in the range [0,1]. -->
           <mean>0.0</mean>
           <stddev>0.007</stddev>
         </noise>
       </camera>
-      <plugin name="camera_controller" filename="libgazebo_ros_camera.so">
+      <camera name="right">
+        <pose>0 -0.16 0 0 0 0</pose>
+        <horizontal_fov>1.3962634</horizontal_fov>
+        <image>
+          <width>800</width>
+          <height>800</height>
+          <format>R8G8B8</format>
+        </image>
+        <clip>
+          <near>0.02</near>
+          <far>300</far>
+        </clip>
+        <noise>
+          <type>gaussian</type>
+          <mean>0.0</mean>
+          <stddev>0.007</stddev>
+        </noise>
+      </camera>
+      <plugin name="stereo_camera_controller" filename="libgazebo_ros_multicamera.so">
         <alwaysOn>true</alwaysOn>
         <updateRate>0.0</updateRate>
-        <cameraName>rrbot/camera1</cameraName>
+        <cameraName>stereo</cameraName>
         <imageTopicName>image_raw</imageTopicName>
         <cameraInfoTopicName>camera_info</cameraInfoTopicName>
-        <frameName>camera_link</frameName>
-        <hackBaseline>0.07</hackBaseline>
+        <frameName>left_cam_rotated</frameName>
+        <rightFrameName>right_cam_rotated</rightFrameName>
+        <hackBaseline>0.16</hackBaseline>
         <distortionK1>0.0</distortionK1>
         <distortionK2>0.0</distortionK2>

Commit message: Added GPS and new urdf configuration

File: urdf/rover1.urdf.xacro (robot description, xacro)
@@ -1,4 +1,4 @@
 <?xml version="1.0"?>
-<robot name="macroed" xmlns:xacro="http://ros.org/wiki/xacro">
+<robot name="paul" xmlns:xacro="http://ros.org/wiki/xacro">
   <xacro:property name="bodywidth" value="0.5" />
   <xacro:property name="bodylen" value="1" />
@@ -27,4 +27,7 @@
     <color rgba="1 1 1 1"/>
   </material>
+  <material name="orange">
+    <color rgba="${255/255} ${108/255} ${10/255} 1.0"/>
+  </material>
   <xacro:macro name="default_inertial" params="mass">
     <inertial>
@@ -45,262 +48,11 @@
       </geometry>
     </collision>
-    <mass value="30" />
+     <xacro:default_inertial mass="30"/>
   </link>
-  <xacro:macro name="wheel" params="prefix suffix reflect length angle parent">
-    <link name="${prefix}_${suffix}_wheel">
-      <visual>
-        <origin xyz="0 0 0" rpy="${pi/2} 0 0" />
-        <geometry>
-          <cylinder radius="${wheeldiam/2}" length="0.1"/>
-        </geometry>
-        <material name="white"/>
-      </visual>
-      <collision>
-        <origin xyz="0 0 0" rpy="${pi/2} 0 0" />
-        <geometry>
-          <cylinder radius="${wheeldiam/2}" length="0.1"/>
-        </geometry>
-      </collision>
-      <xacro:default_inertial mass="1"/>
-    </link>
-    <joint name="${prefix}_${suffix}_wheel_joint" type="continuous">
-      <axis xyz="0 1 0" rpy="0 0 0" />
-      <parent link="${prefix}_${parent}"/>
-      <child link="${prefix}_${suffix}_wheel"/>
-      <origin xyz="${length*sin(angle)} 0 ${-length*cos(angle)}" rpy="0 0 0"/>
-    </joint>
-    <transmission name="${prefix}_${suffix}_wheel_trans">
-      <type>transmission_interface/SimpleTransmission</type>
-      <actuator name="${prefix}_${suffix}_wheel_motor">
-        <mechanicalReduction>1</mechanicalReduction>
-      </actuator>
-      <joint name="${prefix}_${suffix}_wheel_joint">
-        <hardwareInterface>VelocityJointInterface</hardwareInterface>
-      </joint>
-    </transmission>
-    <gazebo reference="${prefix}_${suffix}_wheel">
-      <mu1 value="200.0"/>
-      <mu2 value="100.0"/>
-      <kp value="10000000.0" />
-      <kd value="1.0" />
-      <material>Gazebo/Grey</material>
-    </gazebo>
-  </xacro:macro>
-  <xacro:macro name="rocker_bogie" params="prefix reflect">
-    <link name="${prefix}_rocker_bogie1">
-      <visual>
-        <geometry>
-          <box size="${rocker_bogie_len} ${rocker_thick1} ${rocker_thick2}"/>
-        </geometry>
-        <origin xyz="${sin(rocker2_angle)*rocker_bogie_len/2} 0 ${-cos(rocker2_angle)*rocker_bogie_len/2}" rpy="0  ${rocker1_angle} 0"/>
-        <material name="green"/>
-      </visual>
-      <collision>
-        <geometry>
-          <box size="${rocker_bogie_len} ${rocker_thick1} ${rocker_thick2}"/>
-        </geometry>
-        <origin xyz="${sin(rocker2_angle)*rocker_bogie_len/2} 0 ${-cos(rocker2_angle)*rocker_bogie_len/2}" rpy="0  ${rocker1_angle} 0"/>
-        <material name="green"/>
-      </collision>
-      <xacro:default_inertial mass="1"/>
-    </link>
-    <joint name="rocker_to_${prefix}_rocker_bogie" type="fixed">
-      <parent link="${prefix}_rocker2"/>
-      <child link="${prefix}_rocker_bogie1"/>
-      <origin xyz="${-rocker_len_short*cos(rocker1_angle)} 0 ${-rocker_len_short*sin(rocker1_angle)}" />
-    </joint>
-    <link name="${prefix}_rocker_bogie2">
-       <visual>
-        <geometry>
-          <box size="${rocker_bogie_len} ${rocker_thick1} ${rocker_thick2}"/>
-        </geometry>
-        <origin xyz="${-sin(rocker2_angle)*rocker_bogie_len/2} 0 ${-cos(rocker2_angle)*rocker_bogie_len/2}" rpy="0  ${-rocker1_angle} 0"/>
-        <material name="green"/>
-      </visual>
-      <collision>
-        <geometry>
-          <box size="${rocker_bogie_len} ${rocker_thick1} ${rocker_thick2}"/>
-        </geometry>
-        <origin xyz="${-sin(rocker2_angle)*rocker_bogie_len/2} 0 ${-cos(rocker2_angle)*rocker_bogie_len/2}" rpy="0  ${-rocker1_angle} 0"/>
-        <material name="green"/>
-      </collision>
-      <xacro:default_inertial mass="0.5"/>
-    </link>
-    <joint name="${prefix}_rocker_bogie_joint" type="fixed">
-      <parent link="${prefix}_rocker_bogie1"/>
-      <child link="${prefix}_rocker_bogie2"/>
-      <origin xyz="0 0 0" />
-    </joint>
-    <xacro:wheel prefix="${prefix}" suffix="back" reflect="-1" length="${rocker_bogie_len}" angle="${-rocker1_angle}" parent="rocker_bogie2"/>
-    <xacro:wheel prefix="${prefix}" suffix="middle" reflect="-1" length="${rocker_bogie_len}" angle="${rocker1_angle}" parent="rocker_bogie1"/>
-  </xacro:macro>
-  <xacro:macro name="rocker" params="prefix reflect">
-    <link name="${prefix}_rocker1">
-      <visual>
-        <geometry>
-          <box size="${rocker_len_long+rocker_thick1} ${rocker_thick1} ${rocker_thick2}"/>
-        </geometry>
-        <origin xyz="${sin(rocker1_angle)*rocker_len_long/2} 0 -${cos(rocker1_angle)*rocker_len_long/2}" rpy="0  ${rocker1_angle} 0"/>
-        <material name="green"/>
-      </visual>
-      <collision>
-         <geometry>
-          <box size="${rocker_len_long+rocker_thick1} ${rocker_thick1} ${rocker_thick2}"/>
-        </geometry>
-        <origin xyz="${sin(rocker1_angle)*rocker_len_long/2} 0 -${cos(rocker1_angle)*rocker_len_long/2}" rpy="0  ${rocker1_angle} 0"/>
-      </collision>
-      <xacro:default_inertial mass="0.5"/>
-    </link>
-    <joint name="base_to_${prefix}_rocker" type="fixed">
-      <parent link="base_link"/>
-      <child link="${prefix}_rocker1"/>
-      <origin xyz="0 ${reflect*bodywidth/2} 0" />
-    </joint>
-    <link name="${prefix}_rocker2">
-       <visual>
-        <geometry>
-          <box size="${rocker_len_short+rocker_thick1} ${rocker_thick1} ${rocker_thick2}"/>
-        </geometry>
-        <origin xyz="${-sin(rocker1_angle)*rocker_len_short/2} 0 -${cos(rocker1_angle)*rocker_len_short/2}" rpy="0  ${-rocker1_angle} 0"/>
-        <material name="green"/>
-      </visual>
-      <collision>
-        <geometry>
-          <box size="${rocker_len_short+rocker_thick1} ${rocker_thick1} ${rocker_thick2}"/>
-        </geometry>
-        <origin xyz="${-sin(rocker1_angle)*rocker_len_short/2} 0 -${cos(rocker1_angle)*rocker_len_short/2}" rpy="0  ${-rocker1_angle} 0"/>
-      </collision>
-      <xacro:default_inertial mass="0.5"/>
-    </link>
-    <joint name="${prefix}_rocker_joint" type="fixed">
-      <parent link="${prefix}_rocker1"/>
-      <child link="${prefix}_rocker2"/>
-      <origin xyz="0 0 0" />
-    </joint>
-    <xacro:rocker_bogie prefix="${prefix}" reflect="${reflect}"/>
-    <xacro:wheel prefix="${prefix}" suffix="front" reflect="1" length="${rocker_len_long}" angle="${rocker1_angle}" parent="rocker1"/>
-<!--<xacro:wheel prefix="${prefix}" suffix="front" reflect="1"/>
-    <xacro:wheel prefix="${prefix}" suffix="back" reflect="-1"/> -->
-  </xacro:macro>
-  <xacro:rocker prefix="right" reflect="-1" />
-  <xacro:rocker prefix="left" reflect="1" />
-  <joint name="camera_base_joint" type="fixed">
-    <axis xyz="0 1 0" />
-    <origin xyz="${bodylen/2} 0 0" rpy="0 0 0"/>
-    <parent link="base_link"/>
-    <child link="camera_base_link"/>
-  </joint>
-  <!-- Camera base-->
-  <link name="camera_base_link">
-    <collision>
-      <origin xyz="0 0 0" rpy="0 0 0"/>
-      <geometry>
-    <box size="0.03 0.175 0.033"/>
-      </geometry>
-    </collision>
-    <visual>
-      <origin xyz="0 0 0" rpy="0 0 0"/>
-      <geometry>
-    <box size="0.03 0.175 0.033"/>
-      </geometry>
-      <material name="black"/>
-    </visual>
-    <inertial>
-      <mass value="0.166" />
-      <origin xyz="0 0 0" rpy="0 0 0"/>
-      <inertia ixx="1e-6" ixy="0" ixz="0" iyy="1e-6" iyz="0" izz="1e-6" />
-    </inertial>
-  </link>
-  <!-- Camera -->
-<xacro:macro name="Zedcamera" params="prefix reflect">
-  <joint name="camera_${prefix}_joint" type="fixed">
-    <axis xyz="0 1 0" />
-    <origin xyz="0.015 ${reflect*0.08} 0" rpy="0 0 0"/>
-    <parent link="camera_base_link"/>
-    <child link="camera_${prefix}_link"/>
-  </joint>
-  <link name="camera_${prefix}_link">
-    <collision>
-      <origin xyz="0 0 0" rpy="0 0 0"/>
-      <geometry>
-    <box size="0.01 0.01 0.01"/>
-      </geometry>
-    </collision>
-    <visual>
-      <origin xyz="0 0 0" rpy="0 0 0"/>
-      <geometry>
-    <box size="0.01 0.01 0.01"/>
-      </geometry>
-      <material name="red"/>
-    </visual>
-    <inertial>
-      <mass value="0.166" />
-      <origin xyz="0 0 0" rpy="0 0 0"/>
-      <inertia ixx="1e-6" ixy="0" ixz="0" iyy="1e-6" iyz="0" izz="1e-6" />
-    </inertial>
-  </link>
- </xacro:macro>
-  <xacro:Zedcamera prefix="right" reflect="-1" />
-  <xacro:Zedcamera prefix="left" reflect="1" />
-  <!-- camera -->
-  <gazebo reference="camera_left_link">
-    <sensor type="multicamera" name="stereo_camera">
-      <update_rate>30.0</update_rate>
-      <camera name="left">
-        <horizontal_fov>1.3962634</horizontal_fov>
-        <image>
-          <width>800</width>
-          <height>800</height>
-          <format>R8G8B8</format>
-        </image>
-        <clip>
-          <near>0.02</near>
-          <far>300</far>
-        </clip>
-        <noise>
-          <type>gaussian</type>
-          <mean>0.0</mean>
-          <stddev>0.007</stddev>
-        </noise>
-      </camera>
-      <camera name="right">
-        <pose>0 -0.16 0 0 0 0</pose>
-        <horizontal_fov>1.3962634</horizontal_fov>
-        <image>
-          <width>800</width>
-          <height>800</height>
-          <format>R8G8B8</format>
-        </image>
-        <clip>
-          <near>0.02</near>
-          <far>300</far>
-        </clip>
-        <noise>
-          <type>gaussian</type>
-          <mean>0.0</mean>
-          <stddev>0.007</stddev>
-        </noise>
-      </camera>
-      <plugin name="stereo_camera_controller" filename="libgazebo_ros_multicamera.so">
-        <alwaysOn>true</alwaysOn>
-        <updateRate>0.0</updateRate>
-        <cameraName>stereo</cameraName>
-        <imageTopicName>image_raw</imageTopicName>
-        <cameraInfoTopicName>camera_info</cameraInfoTopicName>
-        <frameName>left_cam_rotated</frameName>
-        <rightFrameName>right_cam_rotated</rightFrameName>
-        <hackBaseline>0.16</hackBaseline>
-        <distortionK1>0.0</distortionK1>
-        <distortionK2>0.0</distortionK2>
-        <distortionK3>0.0</distortionK3>
-        <distortionT1>0.0</distortionT1>
-        <distortionT2>0.0</distortionT2>
-      </plugin>
-    </sensor>
-  </gazebo>
-  <gazebo>
-    <plugin name="gazebo_ros_control" filename="libgazebo_ros_control.so">
-      <robotNamespace>/</robotNamespace>
-    </plugin>
-  </gazebo>
+<!-- Insert Suspensions and wheels -->
+ <xacro:include filename="$(find polyorbite_rover)/urdf/suspensions_wheels.urdf.xacro"/>
+<!-- Insert Camera -->
+ <xacro:include filename="$(find polyorbite_rover)/urdf/camera.urdf.xacro"/>
+<!-- Insert GPS -->
+ <xacro:include filename="$(find polyorbite_rover)/urdf/gps.urdf.xacro"/>
 </robot>

Commit message: Systeme Navigation sans GPS fonctionnel, move_base fonctionnel

File: urdf/rover1.urdf.xacro (robot description, xacro)
@@ -5,5 +5,5 @@
   <xacro:property name="bodyhei" value="0.3" />
   <xacro:property name="wheeldiam" value="0.254" />
-  <xacro:property name="wheellen" value="0.002" />
+  <xacro:property name="wheellen" value="0.001" />
   <xacro:property name="leglen" value="0.6" />
   <xacro:property name="pi" value="3.1415" />

File: urdf/suspensions_wheels.urdf.xacro (robot description, xacro)
@@ -6,5 +6,5 @@
         <origin xyz="0 0 0" rpy="${pi/2} 0 0" />
         <geometry>
-          <cylinder radius="${wheeldiam/2}" length="0.1"/>
+          <cylinder radius="${wheeldiam/2}" length="${wheellen}"/>
         </geometry>
         <material name="white"/>
@@ -13,5 +13,5 @@
         <origin xyz="0 0 0" rpy="${pi/2} 0 0" />
         <geometry>
-          <cylinder radius="${wheeldiam/2}" length="0.1"/>
+          <cylinder radius="${wheeldiam/2}" length="${wheellen}"/>
         </geometry>
        </collision>
@@ -34,13 +34,4 @@
       </joint>
     </transmission>
-    <gazebo reference="${prefix}_${suffix}_wheel">
-	  <mu1 value="100.0"/>
-      <mu2 value="200.0"/>
-      <kp value="1000000.0" />
-      <kd value="100.0" />
-      <!--<maxVel>1.0</maxVel>-->
-	  <minDepth>0.005</minDepth>
-      <material>Gazebo/Grey</material>
-    </gazebo>
   </xacro:macro>
   <xacro:macro name="rocker_bogie" params="prefix reflect">
@@ -113,5 +104,5 @@
       <child link="${prefix}_rocker1"/>
       <origin xyz="0 ${reflect*bodywidth/2} 0" />
-      <!-- <axis xyz="0 1 0" rpy="0 0 0" />
+      <axis xyz="0 1 0" rpy="0 0 0" />
       joint torsional spring plugin <axis>
         <limit>
@@ -136,5 +127,5 @@
           </limit>
         </ode>
-      </physics> -->
+      </physics>
     </joint>
     <link name="${prefix}_rocker2">
